File: 1-4_demux_x2.kicad_sch (KiCad schematic)
At the start: 2 parts, among them U12 74LS139

Commit message: feat: pcb schematic finalization
Parts:
- C15: renamed from C5; value C -> 100n; footprint (none) -> Capacitor_SMD:C_0603_1608Metric_Pad1.08x0.95mm_HandSolder
- U13: renamed from U12; footprint (none) -> Package_SO:SOIC-16_3.9x9.9mm_P1.27mm
Changed lines of the file:
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@@
+	(wire
+		(pts
+			(xy 135.89 45.72) (xy 139.7 45.72)
+		)
+		(stroke
+			(width 0)
+			(type default)
+		)
+	)
 	(wire
 		(pts
@@
 		(pts
 			(xy 148.59 48.26) (xy 152.4 48.26)
+		)
+		(stroke
+			(width 0)
+			(type default)
+		)
+	)
+	(wire
+		(pts
+			(xy 135.89 48.26) (xy 139.7 48.26)
 		)
 		(stroke
@@
 		)
 	)
+	(label "1_X"
+		(at 139.7 45.72 180)
+		(effects
+			(font
+				(size 1.27 1.27)
+			)
+			(justify right bottom)
+		)
+	)
 	(label "1_Y1"
 		(at 181.61 48.26 180)
@@
 	(label "1_Y0"
 		(at 181.61 45.72 180)
+		(effects
+			(font
+				(size 1.27 1.27)
+			)
+			(justify right bottom)
+		)
+	)
+	(label "2_X"
+		(at 139.7 48.26 180)
 		(effects
 			(font
@@
 		(dnp no)
 		(fields_autoplaced yes)
-		(property "Reference" "#PWR020"
+		(property "Reference" "#PWR060"
 			(at 177.8 147.32 0)
 			(hide yes)
@@
 				(path "/2f9d63ef-4408-4e64-a9eb-2669ac711241/03dd6cf7-25a6-43d8-8cf6-4be8b4221c08"
 					(reference "#PWR020")
+					(unit 1)
+				)
+				(path "/2f9d63ef-4408-4e64-a9eb-2669ac711241/3c736a3c-5087-40aa-9b51-da90e91ade5b/77a6507b-9397-4bd1-95b0-60bc2aae4d72"
+					(reference "#PWR064")
+					(unit 1)
+				)
+				(path "/2f9d63ef-4408-4e64-a9eb-2669ac711241/3c736a3c-5087-40aa-9b51-da90e91ade5b/96ed2177-9d3c-41d8-b984-db21da1fdf7e"
+					(reference "#PWR060")
+					(unit 1)
+				)
+				(path "/2f9d63ef-4408-4e64-a9eb-2669ac711241/eefc4e13-3f12-488a-b8ee-fbc666210f78/77a6507b-9397-4bd1-95b0-60bc2aae4d72"
+					(reference "#PWR072")
+					(unit 1)
+				)
+				(path "/2f9d63ef-4408-4e64-a9eb-2669ac711241/eefc4e13-3f12-488a-b8ee-fbc666210f78/96ed2177-9d3c-41d8-b984-db21da1fdf7e"
+					(reference "#PWR071")
 					(unit 1)
 				)
@@
 		(dnp no)
 		(fields_autoplaced yes)
-		(property "Reference" "#PWR019"
+		(property "Reference" "#PWR059"
 			(at 177.8 116.84 0)
 			(hide yes)
@@
 				(path "/2f9d63ef-4408-4e64-a9eb-2669ac711241/03dd6cf7-25a6-43d8-8cf6-4be8b4221c08"
 					(reference "#PWR019")
+					(unit 1)
+				)
+				(path "/2f9d63ef-4408-4e64-a9eb-2669ac711241/3c736a3c-5087-40aa-9b51-da90e91ade5b/77a6507b-9397-4bd1-95b0-60bc2aae4d72"
+					(reference "#PWR063")
+					(unit 1)
+				)
+				(path "/2f9d63ef-4408-4e64-a9eb-2669ac711241/3c736a3c-5087-40aa-9b51-da90e91ade5b/96ed2177-9d3c-41d8-b984-db21da1fdf7e"
+					(reference "#PWR059")
+					(unit 1)
+				)
+				(path "/2f9d63ef-4408-4e64-a9eb-2669ac711241/eefc4e13-3f12-488a-b8ee-fbc666210f78/77a6507b-9397-4bd1-95b0-60bc2aae4d72"
+					(reference "#PWR070")
+					(unit 1)
+				)
+				(path "/2f9d63ef-4408-4e64-a9eb-2669ac711241/eefc4e13-3f12-488a-b8ee-fbc666210f78/96ed2177-9d3c-41d8-b984-db21da1fdf7e"
+					(reference "#PWR069")
 					(unit 1)
 				)
@@
 		(dnp no)
 		(fields_autoplaced yes)
-		(property "Reference" "U12"
+		(property "Reference" "U13"
 			(at 165.1 60.96 0)
 			(show_name no)
@@
 			)
 		)
-		(property "Footprint" ""
+		(property "Footprint" "Package_SO:SOIC-16_3.9x9.9mm_P1.27mm"
 			(at 165.1 71.12 0)
 			(hide yes)
@@
 				(path "/2f9d63ef-4408-4e64-a9eb-2669ac711241/03dd6cf7-25a6-43d8-8cf6-4be8b4221c08"
 					(reference "U12")
+					(unit 2)
+				)
+				(path "/2f9d63ef-4408-4e64-a9eb-2669ac711241/3c736a3c-5087-40aa-9b51-da90e91ade5b/77a6507b-9397-4bd1-95b0-60bc2aae4d72"
+					(reference "U14")
+					(unit 2)
+				)
+				(path "/2f9d63ef-4408-4e64-a9eb-2669ac711241/3c736a3c-5087-40aa-9b51-da90e91ade5b/96ed2177-9d3c-41d8-b984-db21da1fdf7e"
+					(reference "U13")
+					(unit 2)
+				)
+				(path "/2f9d63ef-4408-4e64-a9eb-2669ac711241/eefc4e13-3f12-488a-b8ee-fbc666210f78/77a6507b-9397-4bd1-95b0-60bc2aae4d72"
+					(reference "U16")
+					(unit 2)
+				)
+				(path "/2f9d63ef-4408-4e64-a9eb-2669ac711241/eefc4e13-3f12-488a-b8ee-fbc666210f78/96ed2177-9d3c-41d8-b984-db21da1fdf7e"
+					(reference "U15")
 					(unit 2)
 				)
@@
 		(dnp no)
 		(fields_autoplaced yes)
-		(property "Reference" "U12"
+		(property "Reference" "U13"
 			(at 165.1 38.1 0)
 			(show_name no)
@@
 			)
 		)
-		(property "Footprint" ""
+		(property "Footprint" "Package_SO:SOIC-16_3.9x9.9mm_P1.27mm"
 			(at 165.1 48.26 0)
 			(hide yes)
@@
 				(path "/2f9d63ef-4408-4e64-a9eb-2669ac711241/03dd6cf7-25a6-43d8-8cf6-4be8b4221c08"
 					(reference "U12")
+					(unit 1)
+				)
+				(path "/2f9d63ef-4408-4e64-a9eb-2669ac711241/3c736a3c-5087-40aa-9b51-da90e91ade5b/77a6507b-9397-4bd1-95b0-60bc2aae4d72"
+					(reference "U14")
+					(unit 1)
+				)
+				(path "/2f9d63ef-4408-4e64-a9eb-2669ac711241/3c736a3c-5087-40aa-9b51-da90e91ade5b/96ed2177-9d3c-41d8-b984-db21da1fdf7e"
+					(reference "U13")
+					(unit 1)
+				)
+				(path "/2f9d63ef-4408-4e64-a9eb-2669ac711241/eefc4e13-3f12-488a-b8ee-fbc666210f78/77a6507b-9397-4bd1-95b0-60bc2aae4d72"
+					(reference "U16")
+					(unit 1)
+				)
+				(path "/2f9d63ef-4408-4e64-a9eb-2669ac711241/eefc4e13-3f12-488a-b8ee-fbc666210f78/96ed2177-9d3c-41d8-b984-db21da1fdf7e"
+					(reference "U15")
 					(unit 1)
 				)
@@
 		(dnp no)
 		(fields_autoplaced yes)
-		(property "Reference" "#PWR018"
+		(property "Reference" "#PWR058"
 			(at 152.4 147.32 0)
 			(hide yes)
@@
 				(path "/2f9d63ef-4408-4e64-a9eb-2669ac711241/03dd6cf7-25a6-43d8-8cf6-4be8b4221c08"
 					(reference "#PWR018")
+					(unit 1)
+				)
+				(path "/2f9d63ef-4408-4e64-a9eb-2669ac711241/3c736a3c-5087-40aa-9b51-da90e91ade5b/77a6507b-9397-4bd1-95b0-60bc2aae4d72"
+					(reference "#PWR062")
+					(unit 1)
+				)
+				(path "/2f9d63ef-4408-4e64-a9eb-2669ac711241/3c736a3c-5087-40aa-9b51-da90e91ade5b/96ed2177-9d3c-41d8-b984-db21da1fdf7e"
+					(reference "#PWR058")
+					(unit 1)
+				)
+				(path "/2f9d63ef-4408-4e64-a9eb-2669ac711241/eefc4e13-3f12-488a-b8ee-fbc666210f78/77a6507b-9397-4bd1-95b0-60bc2aae4d72"
+					(reference "#PWR068")
+					(unit 1)
+				)
+				(path "/2f9d63ef-4408-4e64-a9eb-2669ac711241/eefc4e13-3f12-488a-b8ee-fbc666210f78/96ed2177-9d3c-41d8-b984-db21da1fdf7e"
+					(reference "#PWR067")
 					(unit 1)
 				)
@@
 		(dnp no)
 		(fields_autoplaced yes)
-		(property "Reference" "C5"
+		(property "Reference" "C15"
 			(at 156.21 125.7299 0)
 			(show_name no)
@@
 			)
 		)
-		(property "Value" "C"
+		(property "Value" "100n"
 			(at 156.21 128.2699 0)
 			(show_name no)
@@
 			)
 		)
-		(property "Footprint" ""
+		(property "Footprint" "Capacitor_SMD:C_0603_1608Metric_Pad1.08x0.95mm_HandSolder"
 			(at 153.3652 130.81 0)
 			(hide yes)
@@
 				(path "/2f9d63ef-4408-4e64-a9eb-2669ac711241/03dd6cf7-25a6-43d8-8cf6-4be8b4221c08"
 					(reference "C5")
+					(unit 1)
+				)
+				(path "/2f9d63ef-4408-4e64-a9eb-2669ac711241/3c736a3c-5087-40aa-9b51-da90e91ade5b/77a6507b-9397-4bd1-95b0-60bc2aae4d72"
+					(reference "C16")
+					(unit 1)
+				)
+				(path "/2f9d63ef-4408-4e64-a9eb-2669ac711241/3c736a3c-5087-40aa-9b51-da90e91ade5b/96ed2177-9d3c-41d8-b984-db21da1fdf7e"
+					(reference "C15")
+					(unit 1)
+				)
+				(path "/2f9d63ef-4408-4e64-a9eb-2669ac711241/eefc4e13-3f12-488a-b8ee-fbc666210f78/77a6507b-9397-4bd1-95b0-60bc2aae4d72"
+					(reference "C18")
+					(unit 1)
+				)
+				(path "/2f9d63ef-4408-4e64-a9eb-2669ac711241/eefc4e13-3f12-488a-b8ee-fbc666210f78/96ed2177-9d3c-41d8-b984-db21da1fdf7e"
+					(reference "C17")
 					(unit 1)
 				)
@@
 		(dnp no)
 		(fields_autoplaced yes)
-		(property "Reference" "#PWR017"
+		(property "Reference" "#PWR057"
 			(at 152.4 116.84 0)
 			(hide yes)
@@
 				(path "/2f9d63ef-4408-4e64-a9eb-2669ac711241/03dd6cf7-25a6-43d8-8cf6-4be8b4221c08"
 					(reference "#PWR017")
+					(unit 1)
+				)
+				(path "/2f9d63ef-4408-4e64-a9eb-2669ac711241/3c736a3c-5087-40aa-9b51-da90e91ade5b/77a6507b-9397-4bd1-95b0-60bc2aae4d72"
+					(reference "#PWR061")
+					(unit 1)
+				)
+				(path "/2f9d63ef-4408-4e64-a9eb-2669ac711241/3c736a3c-5087-40aa-9b51-da90e91ade5b/96ed2177-9d3c-41d8-b984-db21da1fdf7e"
+					(reference "#PWR057")
+					(unit 1)
+				)
+				(path "/2f9d63ef-4408-4e64-a9eb-2669ac711241/eefc4e13-3f12-488a-b8ee-fbc666210f78/77a6507b-9397-4bd1-95b0-60bc2aae4d72"
+					(reference "#PWR066")
+					(unit 1)
+				)
+				(path "/2f9d63ef-4408-4e64-a9eb-2669ac711241/eefc4e13-3f12-488a-b8ee-fbc666210f78/96ed2177-9d3c-41d8-b984-db21da1fdf7e"
+					(reference "#PWR065")
 					(unit 1)
 				)
@@
 		(dnp no)
 		(fields_autoplaced yes)
-		(property "Reference" "U12"
+		(property "Reference" "U13"
 			(at 184.15 125.7299 0)
 			(show_name no)
@@
 			)
 		)
-		(property "Footprint" ""
+		(property "Footprint" "Package_SO:SOIC-16_3.9x9.9mm_P1.27mm"
 			(at 177.8 127 0)
 			(hide yes)
@@
 					(unit 3)
 				)
+				(path "/2f9d63ef-4408-4e64-a9eb-2669ac711241/3c736a3c-5087-40aa-9b51-da90e91ade5b/77a6507b-9397-4bd1-95b0-60bc2aae4d72"
+					(reference "U14")
+					(unit 3)
+				)
+				(path "/2f9d63ef-4408-4e64-a9eb-2669ac711241/3c736a3c-5087-40aa-9b51-da90e91ade5b/96ed2177-9d3c-41d8-b984-db21da1fdf7e"
+					(reference "U13")
+					(unit 3)
+				)
+				(path "/2f9d63ef-4408-4e64-a9eb-2669ac711241/eefc4e13-3f12-488a-b8ee-fbc666210f78/77a6507b-9397-4bd1-95b0-60bc2aae4d72"
+					(reference "U16")
+					(unit 3)
+				)
+				(path "/2f9d63ef-4408-4e64-a9eb-2669ac711241/eefc4e13-3f12-488a-b8ee-fbc666210f78/96ed2177-9d3c-41d8-b984-db21da1fdf7e"
+					(reference "U15")
+					(unit 3)
+				)
