File: 2-1_mux_x4.kicad_sch (KiCad schematic)
At the start: 4 parts, among them U6 74LS153, U7 74LS153

Commit message: feat: pcb schematic finalization
Parts:
- removed C11, C12: 100n, Capacitor_SMD:C_0603_1608Metric_Pad1.08x0.95mm_HandSolder, symbol Device:C
- removed U6, U7: 74LS153, Package_SO:SOIC-16_3.9x9.9mm_P1.27mm, symbol 74xx:74LS153
- added C26, C27: 100n, Capacitor_SMD:C_0603_1608Metric_Pad1.08x0.95mm_HandSolder, symbol Device:C
- added U22, U23: 74LS153, Package_SO:SOIC-16_3.9x9.9mm_P1.27mm, symbol 74xx:74LS153
Connections:
- net 1_X0: now also U22.6 (I0a)
- net 1_X1: now also U22.10 (I0b)
- net 1_X2: now also U23.6 (I0a)
- net 1_X3: now also U23.10 (I0b)
- net 2_X0: now also U22.5 (I1a)
- net 2_X1: now also U22.11 (I1b)
- net 2_X2: now also U23.5 (I1a)
- net 2_X3: now also U23.11 (I1b)
- net GND: now also C26.2, C27.2, U22.1 (Ea), U22.12 (I2b), U22.13 (I3b), U22.15 (Eb), U22.2 (S1), U22.3 (I3a), U22.4 (I2a), U22.8 (GND), U23.1 (Ea), U23.12 (I2b), U23.13 (I3b), U23.15 (Eb), U23.2 (S1), U23.3 (I3a), U23.4 (I2a), U23.8 (GND)
- net S0: now also U22.14 (S0), U23.14 (S0)
- net VDD: now also C26.1, C27.1, U22.16 (VCC), U23.16 (VCC)
- net Y0: now also U22.7 (Za)
- net Y1: now also U22.9 (Zb)
- net Y2: now also U23.7 (Za)
- net Y3: now also U23.9 (Zb)
